File: pcb_peau_v1/_autosave-pcb_peau_v1.kicad_pcb (KiCad board)
At the start: 2 copper layers, 76 x 74 mm, 25 parts, among them J1 Conn_01x05, J2 Conn_01x05, J4 Conn_02x08_Top_Bottom, J5 Conn_02x12_Top_Bottom, U2 TLC274, U3 CD74HC4067SM, U4 CD74HC4067SM, U5 CD74HC4067SM, U6 CD74HC4067SM, U7 TLC274, U8 TLC274, U9 TLC274

Commit message: PCB FINI
Routing:
- net 0: track 20.2 -> 43.1 mm, vias 0 -> 4
- net NE2: track 58.6 -> 74.1 mm, vias 2 -> 3
- net +5V: track 181.3 -> 188.7 mm
- net +12V: track 55.3 -> 60.8 mm, vias 0 -> 1
- net AOP2: track 64.4 -> 66.0 mm
- net Net-(J4-Pin_3): track 88.8 -> 90.2 mm, vias 0 -> 2
- net Net-(J4-Pin_5): vias 1 -> 3
- net AOP1: vias 2 -> 4
- net 2-ENTREE: vias 0 -> 1
